Commit message: fixed orientation problem

File: tortoisebot_rtab_mapping/urdf/tortoisebot_w_kinect_v1.xacro (robot description, xacro)
@@ -45,4 +45,5 @@
 		</collision>
 	</link>
+	<link name="camera_frame_optical"/>
 	<joint name="Rigid10" type="fixed">
 		<origin rpy="0 0 0" xyz="0.0 0.0 0.25" />
@@ -55,3 +56,8 @@
 		<child link="kinect_sensor" />
 	</joint>
+	<joint name="camera_optical_joint" type="fixed">
+		<origin xyz="0 0 0" rpy="-1.5708 0 -1.5708"/>
+        <parent link="kinect_sensor"/>
+        <child link="camera_frame_optical"/>
+    </joint>
 </robot>
